File: KiCad/4-Bit_ALU.kicad_pcb (KiCad board)
At the start: 2 copper layers, 106.7 x 134.6 mm, 31 parts, among them U1 74HC86, U10 74LS153, U11 74LS153, U12 4002, U2 74LS08, U3 74HC86, U4 74HC86, U5 74LS08, U6 74HC86, U7 74HC00, U8 74HC86, U9 74HC02

Commit message: Update README and replace Gerber file for 4-Bit ALU project
Parts:
- removed Flags1: Conn_01x02, Connector_PinHeader_2.54mm:PinHeader_1x02_P2.54mm_Vertical
- added J1: EQ Z C, Connector_PinHeader_2.54mm:PinHeader_1x03_P2.54mm_Vertical, F.Cu at (151.1, 107.1)
Connections:
- net Net-(Power1-Pin_1) renamed +5V
- U6 pad 11: unconnected-(U6-Pad11) -> Net-(J1-Pin_3)
Routing:
- net Net-(J1-Pin_3): track 0.00 -> 130.6 mm, vias 0 -> 3
- net Net-(Nibble_B1-Pin_3): track 164.9 -> 166.4 mm
Other:
- board text added: "C ZR EQ"
- board text added: "Hardware-Minimalist 4-bit ALU Modified 3-bit OP Code | Rev 3.3 Made by: Neowizen"
- board text removed: "Hardware-Minimalist 4-bit ALU Modified 3-bit OP Code | Rev 3.2 Made by: Neowizen"
- board text removed: "ZR EQ"
