File: KiCad/4-Bit_ALU.kicad_sch (KiCad schematic)
At the start: 31 parts, among them U1 74HC86, U10 74LS153, U11 74LS153, U12 4002, U2 74LS08, U3 74HC86, U4 74HC86, U5 74LS08, U6 74HC86, U7 74HC00, U8 74HC86, U9 74HC02

Commit message: Update README and replace Gerber file for 4-Bit ALU project
Parts:
- removed Flags1: Conn_01x02, Connector_PinHeader_2.54mm:PinHeader_1x02_P2.54mm_Vertical, symbol Connector_Generic:Conn_01x02
- added J1: EQ Z C, Connector_PinHeader_2.54mm:PinHeader_1x03_P2.54mm_Vertical, symbol Connector_Generic:Conn_01x03
Connections:
- net +5V: now reaches C1.1, C10.1, C11.1, C12.1, C2.1, C3.1, C4.1, C5.1, C6.1, C7.1, C8.1, C9.1, C_Power1.1, Power1.1 (Pin_1), U1.14 (VCC), U10.16 (VCC), U11.16 (VCC), U12.14 (VDD), U2.14 (VCC), U3.14 (VCC), U4.14 (VCC), U5.14 (VCC), U6.14 (VCC), U7.14 (VCC), U8.14 (VCC), U9.14 (VCC)
- net at U12.13: now also J1.1 (Pin_1)
- net at U12.1: now also J1.2 (Pin_2)
- net at U6.11: now also J1.3 (Pin_3)
- no-connect marks 1 -> 0
Other:
- company: Yamil-Serrano -> Neowizen
- moved on the sheet: C1, C10, C11, C12, C2, C3, C4, C5, C6, C7, C8, C9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
